Commit message: Added RGBD Camera

File: src/lerobot_description/urdf/so101_base.xacro (robot description, xacro)
@@ -447,3 +447,33 @@
 		</actuator>
 	</transmission>
+    <link name="camera_link">
+      <visual>
+        <geometry>
+          <box size="0.02 0.05 0.02"/>
+        </geometry>
+        <material name="blue">
+          <color rgba="0 0 1 1"/>
+        </material>
+      </visual>
+      <collision>
+        <geometry>
+          <box size="0.02 0.05 0.02"/>
+        </geometry>
+      </collision>
+      <inertial>
+        <mass value="0.05"/>
+        <inertia ixx="0.0001" ixy="0" ixz="0" iyy="0.0001" iyz="0" izz="0.0001"/>
+      </inertial>
+    </link>
+    <joint name="camera_joint" type="fixed">
+      <parent link="base"/>
+      <child link="camera_link"/>
+       <origin xyz="0 -0.3 1" rpy="0 1.57079632679 0"/>
+    </joint>
+    <link name="camera_link_optical"></link>
+    <joint name="camera_link_optical_joint" type="fixed">
+      <parent link="camera_link"/>
+      <child link="camera_link_optical"/>
+      <origin xyz="0 0 0" rpy="-1.57079632679 0 -1.57079632679"/>
+    </joint>
 </robot>

File: src/lerobot_description/urdf/so101_gazebo.xacro (robot description, xacro)
@@ -6,4 +6,46 @@
             <parameters>$(find lerobot_controller)/config/so101_controllers.yaml</parameters>
         </plugin>
+        <!-- Sensors system plugin - required for camera sensors in Gazebo Harmonic -->
+        <plugin filename="gz-sim-sensors-system" name="gz::sim::systems::Sensors">
+            <render_engine>ogre2</render_engine>
+        </plugin>
+    </gazebo>
+    <gazebo reference="camera_link">
+        <sensor name="camera" type="camera">
+            <always_on>1</always_on>
+            <update_rate>30</update_rate>
+            <topic>camera</topic>
+            <camera name="camera">
+                <horizontal_fov>1.047</horizontal_fov>
+                <image>
+                    <width>640</width>
+                    <height>480</height>
+                    <format>R8G8B8</format>
+                </image>
+                <clip>
+                    <near>0.1</near>
+                    <far>10</far>
+                </clip>
+            </camera>
+        </sensor>
+    </gazebo>
+    <gazebo reference="camera_link">
+        <sensor name="camera_depth" type="depth_camera">
+            <always_on>1</always_on>
+            <update_rate>30</update_rate>
+            <topic>camera_depth</topic>
+            <camera name="camera_depth">
+                <horizontal_fov>1.047</horizontal_fov>
+                <image>
+                    <width>640</width>
+                    <height>480</height>
+                    <format>L8</format>
+                </image>
+                <clip>
+                    <near>0.1</near>
+                    <far>10</far>
+                </clip>
+            </camera>
+        </sensor>
     </gazebo>
 </robot>
